File: kicad/diagral-uart-esp32.kicad_pcb (KiCad board)
At the start: 2 copper layers, 69 x 43 mm, 11 parts, among them J1 DIAGRAL_CONN, U1 XIAO-ESP32-S3, U2 WIZ850io

Commit message: add compatibility with Waveshare ESP32-C6 and Waveshare ESP32-S3 - update PCB to version 1.1
Parts:
- added D2: 1N5819, Diode_THT:D_DO-41_SOD81_P10.16mm_Horizontal, B.Cu at (118.6, 111.5)
- D1: value XL74610 -> 1N5819; footprint my_library:XL74610 -> Diode_THT:D_DO-41_SOD81_P10.16mm_Horizontal
- U1: value XIAO-ESP32-S3 -> Waveshare-ESP32-C6-Zero; footprint my_library:XIAO-ESP32-S3-DIP_batt -> my_library:Waveshare-ESP32-C6-Zero
- moved R6 5.03 mm to (161.0, 117.1), turned to 90 degrees
- moved D1 4.69 mm to (118.6, 99.5)
- moved R5 3.42 mm to (169.0, 110.5)
- moved BT1 2.50 mm to (167.4, 102.0)
- moved U1 1.46 mm to (145.5, 106.5), turned to 90 degrees
Connections:
- U1 pad 1: /W5500_RST -> Net-(D1-K)
- U1 pad 10: /Vbat_monitor -> /W5500_INT
- U1 pad 11: unconnected-(U1-D10-Pad11)_1 -> /W5500_CS
- U1 pad 12: +3V3 -> /W5500_SCLK
- U1 pad 13: GND -> /W5500_MOSI
- U1 pad 14: Net-(D1-K) -> /W5500_MISO
- U1 pad 15: +BATT -> /W5500_RST
- U1 pad 16: GND -> /ESP32_SIG
- U1 pad 2: /W5500_MISO -> GND
- U1 pad 3: /W5500_MOSI -> +3V3
- U1 pad 4: /W5500_SCLK -> /Vbat_monitor
- U1 pad 5: /W5500_CS -> unconnected-(U1-IO1-Pad5)
- U1 pad 6: /W5500_INT -> unconnected-(U1-IO2-Pad6)
- U1 pad 7: /ESP32_TX -> unconnected-(U1-IO3-Pad7)
- U1 pad 8: /DIAGRAL_TX -> unconnected-(U1-IO4-Pad8)
- U1 pad 9: /ESP32_SIG -> unconnected-(U1-IO5-Pad9)
Routing:
- net +BATT: track 49.6 -> 100.9 mm, vias 1 -> 0
- net /ESP32_TX: track 6.02 -> 35.6 mm
- net /Vbat_monitor: track 39.6 -> 15.8 mm
- net Net-(D1-K): track 14.1 -> 34.4 mm
- net /W5500_SCLK: track 38.4 -> 58.0 mm
- net /W5500_CS: track 38.7 -> 57.8 mm
- net /W5500_INT: track 39.3 -> 57.7 mm
- net /W5500_MOSI: track 37.9 -> 55.4 mm
- net /W5500_RST: track 14.3 -> 31.7 mm
- net /W5500_MISO: track 15.2 -> 30.8 mm
- net /DIAGRAL_5V: track 60.8 -> 76.2 mm
- net /DIAGRAL_TX: track 55.2 -> 68.5 mm
- net /DIAGRAL_RX: track 33.1 -> 45.8 mm
- net /ESP32_SIG: track 31.5 -> 43.3 mm, vias 0 -> 1
- net +3V3: track 34.9 -> 29.3 mm
Other:
- board text added: "V1.1"
- board text removed: "V1.0"
