File: kicad/diagral-uart-esp32.kicad_sch (KiCad schematic)
At the start: 11 parts, among them J1 DIAGRAL_CONN, U1 XIAO-ESP32-S3, U2 WIZ850io

Commit message: add compatibility with Waveshare ESP32-C6 and Waveshare ESP32-S3 - update PCB to version 1.1
Parts:
- removed D1: XL74610, my_library:XL74610, symbol My symboles:XL74610
- added D1, D2: 1N5819, Diode_THT:D_DO-41_SOD81_P10.16mm_Horizontal, symbol Diode:1N5819
- U1: value XIAO-ESP32-S3 -> Waveshare-ESP32-C6-Zero; footprint my_library:XIAO-ESP32-S3-DIP_batt -> my_library:Waveshare-ESP32-C6-Zero; symbol My symboles:XIAO-ESP32-S3-SMD -> My symboles:Waveshare-ESP32-C6-Zero
Connections:
- net +3V3: now also U1.3 (3V3); no longer U1.12 (3V3_OUT)
- net +BATT: now also D2.2 (A); no longer U1.15 (VBAT)
- net DIAGRAL_5V: now also D1.2 (A)
- net DIAGRAL_TX: now also U1.17 (RX); no longer U1.8 (D7)
- net ESP32_SIG: now also U1.16 (IO14); no longer U1.9 (D8)
- net ESP32_TX: now also U1.18 (TX); no longer U1.7 (D6)
- net GND: now also U1.2 (GND); no longer U1.13 (GND), U1.16 (GND)
- net Vbat_monitor: now also U1.4 (IO0); no longer U1.10 (D9)
- net W5500_CS: now also U1.11 (IO21); no longer U1.5 (D4)
- net W5500_INT: now also U1.10 (IO22); no longer U1.6 (D5)
- net W5500_MISO: now also U1.14 (IO18); no longer U1.2 (D1)
- net W5500_MOSI: now also U1.13 (IO19); no longer U1.3 (D2)
- net W5500_RST: now also U1.15 (IO15); no longer U1.1 (D0)
- net W5500_SCLK: now also U1.12 (IO20); no longer U1.4 (D3)
- new net: D1.1 (K), D2.1 (K), U1.1 (VCC)
- no-connect marks 8 -> 7
Other:
- moved on the sheet: BT1, R1, R2, R5, R6, U2
